Commit message: first commit

File: src/robot_5a_urdf/description/physics_include.xacro (robot description, xacro)
@@ -11,4 +11,7 @@
     <material name="blue">
         <color rgba="0.2 0.2 1 1"/>
+    </material>
+    <material name="green">
+        <color rgba="0.2 1 0.2 1"/>
     </material>
     <!-- Specify some standard inertial calculations https://en.wikipedia.org/wiki/List_of_moments_of_inertia -->

File: src/robot_5a_urdf/description/robot_5a_moveoBCN3D.urdf (robot description, URDF)
Before this commit: robot robot_5a_urdf, 7 links, 6 joints
Links:
- link Link_1: mass 14.597 -> 4.2526
- link Link_2: mass 14.597154271183 -> 1.9323
- link Link_3: mass 14.597154271183 -> 1.1381
- link Link_4: mass 14.597154271183 -> 0.62964
- link Link_5: mass 14.597154271183 -> 0.19875
- link base_link: mass 14.597154271183 -> 8.0643
Joints:
- joint Joint_1: limit lower=-1.5707 upper=1.5707 effort=5 velocity=1 -> lower=-1.5707 upper=1.5707 effort=100 velocity=100
- joint Joint_2: limit lower=-1.5707 upper=1.5707 effort=5 velocity=1 -> lower=-1.5707 upper=1.5707 effort=100 velocity=100
- joint Joint_3: limit lower=-1.5707 upper=1.5707 effort=5 velocity=1 -> lower=-1.5707 upper=1.5707 effort=100 velocity=100
- joint Joint_4: limit lower=-1.5707 upper=1.5707 effort=5 velocity=1 -> lower=-1.5707 upper=1.5707 effort=100 velocity=100
- joint Joint_5: limit lower=-1.5707 upper=1.5707 effort=5 velocity=1 -> lower=-1.5707 upper=1.5707 effort=100 velocity=100

File: src/robot_5a_urdf/description/simulation_gazebo.xacro (robot description, xacro)
@@ -6,23 +6,41 @@
     <!-- Gazebo is unable to use the same <material> tags that are already in the URDF (that RViz uses). -->
     <!-- Instead, we need to add gazebo tags for our links that refer to Gazebo materials -->
-<!--    <gazebo reference="base_link">
+    <gazebo reference="base_link">
         <material>Gazebo/Green</material>
     </gazebo>
-    <gazebo reference="slider_link">
+    <gazebo reference="Link_1">
         <material>Gazebo/Blue</material>
     </gazebo>
-    <gazebo reference="arm_link">
+    <gazebo reference="Link_2">
         <material>Gazebo/Orange</material>
     </gazebo>
--->
+    <gazebo reference="Link_3">
+        <material>Gazebo/Green</material>
+    </gazebo>
+    <gazebo reference="Link_4">
+        <material>Gazebo/BLue</material>
+    </gazebo>
+    <gazebo reference="Link_5">
+        <material>Gazebo/Orange</material>
+    </gazebo>
+    <!-- Fictions
+    <gazebo reference="front_caster">
+        <mu1>0.01</mu1>
+        <mu2>0.01</mu2>
+        <material>Gazebo/White</material>
+        <gravity>true</gravity>
+    </gazebo>
+    -->
     <!-- Gazebo requires the use of plugins to interact with other systems such as ROS. -->
     <!-- This plugin will publish the joint_states for the selected joints
             (which robot_state_publisher can then use to broadcast the approprate tf). -->
     <gazebo>
-        <plugin name="gazebo_ros_joint_state_publisher"
-            filename="libgazebo_ros_joint_state_publisher.so">
+        <plugin name="gazebo_ros_joint_state_publisher" filename="libgazebo_ros_joint_state_publisher.so">
             <update_rate>20</update_rate>
-            <joint_name>slider_joint</joint_name>
-            <joint_name>arm_joint</joint_name>
+            <joint_name>Joint_1</joint_name>
+            <joint_name>Joint_2</joint_name>
+            <joint_name>Joint_3</joint_name>
+            <joint_name>Joint_4</joint_name>
+            <joint_name>Joint_5</joint_name>
         </plugin>
     </gazebo>
@@ -44,4 +62,5 @@
             look at https://www.ros.org/reps/rep-0103.html#suffix-frames for slightly more information. -->
     <!-- First, create the link and joint for the optical frame -->
+    <!--
     <joint name="camera_optical_joint" type="fixed">
         <origin xyz="0 0 0" rpy="-1.571 0 -1.571" />
@@ -50,4 +69,5 @@
     </joint>
     <link name="camera_link_optical"></link>
+-->
     <!-- Add a gazebo tag for the ORIGINAL camera_link (but in the plugin we reference the optical frame so that ROS can orient things correctly) -->
     <!-- Within the gazebo tag we have the sensor tag, and inside that there is (among other things) the camera tag with the camera parameters,
@@ -55,6 +75,6 @@
     <!-- Note that although visualise is set to true, it won't actually visualise the depth camera in gazebo. To see the preview,
             try swapping "depth" to "camera"-->
-            <!---->
-            <gazebo reference="camera_link">
+            <!--
+    <gazebo reference="camera_link">
         <sensor type="depth" name="my_camera">
             <update_rate>20</update_rate>
@@ -84,3 +104,4 @@
         </sensor>
     </gazebo>
+    -->
 </robot>
